File: Hardware/SparkFun_ESP32_Power_Control_Shield.brd (EAGLE design)
At the start: 101.6 x 50.8 mm, 68 parts, among them IC1 LMV358, IC2 LMV358, J2 POWER_JACKPTH_LOCK, U1 MC33926, U2 MC33926, U3 MC33926, U4 R-78E5.0-1.0

Commit message: Replaced R13
Pull down resistor R13 was too weak for the ESP32 at 10k. Replacing with
1k.
Parts:
- R13: value 10k -> 1k
Changed lines of the file:
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@@
 <attribute name="PROD_ID" value="CONN-08288" x="50.8" y="46.99" size="1.778" layer="28" font="vector" ratio="15" rot="MR180" display="off"/>
 </element>
-<element name="R13" library="SparkFun-Resistors" package="0603" value="10k" x="34.798" y="25.908" rot="R270">
-<attribute name="PROD_ID" value="RES-00824" x="34.798" y="25.908" size="1.778" layer="27" font="vector" ratio="15" rot="R270" display="off"/>
+<element name="R13" library="SparkFun-Resistors" package="0603" value="1k" x="34.798" y="25.908" rot="R270">
+<attribute name="PROD_ID" value="RES-07856" x="34.798" y="25.908" size="1.778" layer="27" font="vector" ratio="15" rot="R270" display="off"/>
 </element>
 <element name="R10" library="SparkFun-Resistors" package="AXIAL-0.3" value="" x="40.005" y="17.78" rot="R180">
